Commit message: Change tello camera gazeo

File: tello_description/urdf/quadrotor_with_cam.urdf.xacro (robot description, xacro)
@@ -7,5 +7,5 @@
     <xacro:quadrotor_base_macro />
     <!-- Forward facing camera -->
-    <xacro:include filename="$(find hector_sensors_description)/urdf/generic_camera.urdf.xacro" />
+    <xacro:include filename="$(find tello_description)/urdf/tello_camera.urdf.xacro" />
     <xacro:generic_camera name="front_cam" parent="base_link" ros_topic="camera/image" cam_info_topic="camera/camera_info" update_rate="10" res_x="960" res_y="720" image_format="R8G8B8" hfov="83">
       <origin xyz="0.05 0.0 0.02" rpy="0 0 0"/>

File: tello_description/urdf/tello.urdf.xacro (robot description, xacro)
@@ -26,5 +26,5 @@
     <!-- Sonar height sensor -->
     <xacro:sonar_sensor name="sonar" parent="base_link" ros_topic="sonar_height" update_rate="10" min_range="0.03" max_range="3.0" field_of_view="${40*pi/180}" ray_count="3">
-      <origin xyz="-0.16 0.0 0.12" rpy="0 ${90*pi/180} 0"/>
+      <origin xyz="-0.01 0.0 0.005" rpy="0 ${90*pi/180} 0"/>
     </xacro:sonar_sensor>
   </xacro:macro>
