Commit message: Change mass of tello

File: tello_description/urdf/tello.urdf.xacro (robot description, xacro)
@@ -7,5 +7,5 @@
     <link name="base_link">
       <inertial>
-        <mass value="1.477" />
+        <mass value="0.085" />
         <origin xyz="0 0 0" />
         <inertia ixx="0.01152" ixy="0.0" ixz="0.0" iyy="0.01152" iyz="0.0" izz="0.0218" />
